File: cantact.kicad_pcb (KiCad board)
At the start: 2 copper layers, 36 x 61.1 mm, 38 parts, among them P1 USB, P2 SWD, P3 DB9, U1 STM32F042C6T6, U2 AAT3221, U3 MCP2551-I/SN, X1 16 MHz

Commit message: hardware v0.3, added mounting holes and text
Parts:
- added ?: VAL**, Mounting_Holes:MountingHole_2-5mm, F.Cu at (152.7, 148.3)
- added ?: VAL**, Mounting_Holes:MountingHole_2-5mm, F.Cu at (128.4, 116.5)
- moved C10 3.55 mm to (135.0, 116.3), turned to 0 degrees
- moved R3 1.46 mm to (129.4, 129.3)
Routing:
- net GND: track 225.9 -> 212.1 mm
- net +5V: track 46.9 -> 50.0 mm
- net Net-(D2-Pad2): track 1.99 -> 1.28 mm
Other:
- net class Mounting Hole added: clearance 0.5, trace_width 0.2032, via_dia 6.5, via_drill 3.5
- board text added: "CANtact V0.3"
- board text added: "Eric Evenchick eric@evenchick.com"
- board text added: "http://cantact.io"
- board text added: "http://evenchick.com @ericevenchick"
- board text removed: "CANtact V0.2"

Commit message: final v1.0 fixes, added assembly files
Other:
- board text added: "2 5"
- board text added: "A"
- board text added: "CANtact V1.0"
- board text removed: "5 2"
- board text removed: "CANtact V0.3"
- board text removed: "Eric Evenchick eric@evenchick.com"
- board text removed: "http://evenchick.com @ericevenchick"
